Commit message: burger_desc: add camera with mountplate

File: turtlebot3_description/urdf/turtlebot3_burger.urdf.xacro (robot description, xacro)
@@ -3,4 +3,14 @@
   <xacro:include filename="$(find turtlebot3_description)/urdf/common_properties.xacro"/>
   <xacro:include filename="$(find turtlebot3_description)/urdf/turtlebot3_burger.gazebo.xacro"/>
+  <xacro:include filename="$(find turtlebot3_description)/urdf/mountplate.urdf.xacro"/>
+  <xacro:include filename="$(find turtlebot3_description)/urdf/camera.urdf.xacro"/>
+  <xacro:property name="camera_x_size" value="0.04" />
+  <xacro:property name="camera_y_size" value="0.16" />
+  <xacro:property name="camera_z_size" value="0.03" />
+  <xacro:property name="camera_pitch" value="0" />
+  <xacro:property name="camera_roll" value="-1.57" />
+  <xacro:property name="camera_yaw" value="1.57" />
+  <xacro:property name="camera_mountplate_z_offset" value="0.0" />
+  <xacro:property name="camera_mass" value="0.3" />
   <link name="base_footprint"/>
   <joint name="base_joint" type="fixed">
